File: dual-edge-wake/dual-edge-wake.kicad_pcb (KiCad board)
At the start: 2 copper layers, 16 parts, among them J1 Conn_01x03_Male, J2 Conn_01x02_Male, J3 Conn_01x02_Male, Q1 BC807, Q2 BC847, Q3 BC847, U1 SN74LVC1G86DBVR

Commit message: Finished first PCB
Parts:
- added J4: Leading, Jumper:SolderJumper-2_P1.3mm_Open_RoundedPad1.0x1.5mm, F.Cu at (101.8, 58.0)
- J1: value Conn_01x03_Male -> Conn_01x04_Male; footprint Jumper:SolderJumper-3_P1.3mm_Open_RoundedPad1.0x1.5mm -> Connector_PinHeader_2.54mm:PinHeader_1x04_P2.54mm_Vertical
- J2: value Conn_01x02_Male -> Circuit; footprint Jumper:SolderJumper-2_P1.3mm_Open_RoundedPad1.0x1.5mm -> Jumper:SolderJumper-3_P1.3mm_Open_RoundedPad1.0x1.5mm
- J3: value Conn_01x02_Male -> Falling
- R1, R2, R3, R4, R5, R6: footprint Resistor_SMD:R_0603_1608Metric_Pad0.98x0.95mm_HandSolder -> Resistor_SMD:R_0805_2012Metric_Pad1.20x1.40mm_HandSolder
- moved Q3 58.5 mm to (95.1, 66.5), turned to 180 degrees
- moved R4 49.6 mm to (116.3, 54.1), turned to -90 degrees
- moved J2 49.1 mm to (95.4, 51.6)
- moved R6 49.1 mm to (107.5, 64.3), turned to 90 degrees
- moved C3 47.7 mm to (105.3, 64.3)
- moved R1 47.6 mm to (105.6, 55.9)
- moved R2 45.6 mm to (108.6, 54.0), turned to -90 degrees
- moved U1 45.5 mm to (111.0, 64.3)
- moved J1 45.3 mm to (95.3, 55.2), turned to 0 degrees
- moved Q1 44.3 mm to (112.5, 54.1)
- moved C1 44.1 mm to (105.6, 53.8)
- moved R5 43.5 mm to (116.3, 57.9), turned to 90 degrees
- moved J3 38.3 mm to (101.8, 53.8)
- moved Q2 36.5 mm to (112.5, 57.8)
- moved C2 35.9 mm to (105.6, 58.1)
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Connections:
- net /OutputA renamed /C
- J1 pad 1: /InputA -> +3.3V
- J1 pad 2: /Sensor -> GND
- J1 pad 3: /InputB -> /Input
- J2 pad 1: /InputA -> /A
- J2 pad 2: Net-(C1-Pad1) -> /Input
- J3 pad 1: /InputA -> /A
- J3 pad 2: Net-(C2-Pad1) -> Net-(C1-Pad1)
- R1 pad 2: /InputA -> /A
- R6 pad 2: /InputB -> /B
- U1 pad 1: /InputB -> /B
Routing:
- net /C: track 0.00 -> 53.7 mm
- net +3.3V: track 0.00 -> 44.9 mm, vias 0 -> 3
- net GND: track 0.00 -> 34.0 mm
- net /B: track 0.00 -> 22.8 mm
- net /A: track 0.00 -> 22.6 mm
- net /Input: track 0.00 -> 10.0 mm
- net Net-(C3-Pad2): track 0.00 -> 5.45 mm
- net Net-(R4-Pad2): track 0.00 -> 5.25 mm
- net Net-(C1-Pad2): track 0.00 -> 5.05 mm
- net Net-(C2-Pad2): track 0.00 -> 4.86 mm
- net /Output: track 0.00 -> 4.45 mm
- net Net-(R5-Pad2): track 0.00 -> 2.69 mm
- net Net-(C2-Pad1): track 0.00 -> 2.09 mm
- net Net-(C1-Pad1): track 0.00 -> 2.07 mm
Other:
- board outline added: 28.7 x 22.1 mm
- board text added: "A"
- board text added: "A: Dual edge monostable trigger"
- board text added: "B"
- board text added: "B: Edge to glitch XOR delay"
- board text added: "OUT IN GND VCC"
